File: Hardware/MADC_ARTY/Gain.kicad_sch (KiCad schematic)
At the start: 25 parts, among them U11 AQY212G3HS, U12 AQY212G3HS, U13 ADA4627-1ARZ, U14 AD8422ARMZ

Commit message: GERBER
Parts:
- U14: value AD8422ARMZ -> AD8422ARZ
Changed lines of the file:
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@@
 			)
 		)
-		(property "Value" "AD8422ARMZ"
+		(property "Value" "AD8422ARZ"
 			(at 179.832 102.616 0)
 			(effects
