File: Hardware/MADC_ARTY/MADC_ARTY.kicad_pcb (KiCad board)
At the start: 4 copper layers, 133 x 70 mm, 251 parts, among them J1 FCR7350R, J2 FCR7350B, J3 1715721, J4 71764-0012, J5 71764-0012, Q1 JFE2140DR, Q10 MMBT6429LT1G, Q11 MMBT6429LT1G, Q12 MMBF4392LT1G, Q13 MMBT6429LT1G, Q14 MMBT6429LT1G, Q2 MMBT6429LT1G, Q3 MMBT6429LT1G, Q4 MMBF4392LT1G, Q5 MMBT6429LT1G, Q6 MMBT6429LT1G, Q7 SiS443DN, Q8 MMBT3904VL, Q9 JFE2140DR, U1 ADA4622-4ACPZ, U10 ADP7182ACPZN, U11 AQY212G3HS, U12 AQY212G3HS, U13 ADA4627-1ARZ, U14 AD8422ARMZ, U15 ADG419BRMZ, U16 ADG419BRMZ, U17 MADC (2x62330821021), U18 SN74LVC1T45DBV, U19 OPA2192IDGKT, U2 OP27GSZ, U20 OPA2192IDGKT, U21 ADR1399KHZ, U22 ADR1399KEZ, U23 ADG419BRMZ, U24 ADG419BRMZ, U25 ADA4622-4ACPZ, U26 OP27GSZ, U3 TSR3-2450N, U4 ADP5071AREZ, U5 ADP7142ACPZN, U6 ADP7142ARDZ-3.3, U7 ADP7182ACPZN, U8 ADP7142ARDZ, U9 ADP7182ACPZN

Commit message: GERBER
Parts:
- R70: value 2k7/1%/250mW -> 1k8/1%/250mW
- U10, U7, U9: value ADP7182ACPZN -> ADP7182ACPZN-R7
- U14: value AD8422ARMZ -> AD8422ARZ
- U19, U20: value OPA2192IDGKT -> OPA2192IDR
- U5: value ADP7142ACPZN -> ADP7142ARDZ-R7; footprint Package_CSP:LFCSP-6-1EP_2x2mm_P0.65mm_EP1x1.6mm -> Package_SO:SOIC-8-1EP_3.9x4.9mm_P1.27mm_EP2.29x3mm
- U8: value ADP7142ARDZ -> ADP7142ARDZ-R7
- moved R19 8.02 mm to (113.7, 53.2), turned to -90 degrees
- moved C17 6.65 mm to (111.6, 50.8), turned to -90 degrees
- moved R18 4.04 mm to (113.7, 50.2), turned to -90 degrees
- moved U5 3.54 mm to (118.7, 50.3), turned to 0 degrees
- moved C13 2.75 mm to (120.1, 46.4), turned to 180 degrees
- moved R91 2.01 mm to (116.3, 45.3)
Connections:
- R18 pad 2: Net-(U5-ADJ) -> Net-(U5-SENSE/ADJ)
- R19 pad 1: Net-(U5-ADJ) -> Net-(U5-SENSE/ADJ)
- U5 pad 2: Net-(U5-ADJ) -> +16V
- U5 pad 3: GND -> Net-(U5-SENSE/ADJ)
- U5 pad 4: +18V -> GND
- U5 pad 5: unconnected-(U5-SS-Pad5) -> +18V
- U5 pad 6: +18V -> unconnected-(U5-SS-Pad6)
- U5 pad 7: GND -> +18V
Routing:
- net Net-(U5-SENSE/ADJ): track 0.00 -> 4.03 mm
- net +18V: track 194.6 -> 190.7 mm
- net Net-(U5-ADJ): track 3.16 -> 0.00 mm
- net -18V: track 180.9 -> 182.8 mm
- net -14V: track 56.9 -> 58.1 mm
- net GND: vias 110 -> 111
- net +16V: vias 23 -> 24
