File: Hardware/MADC_ARTY/Power.kicad_sch (KiCad schematic)
At the start: 90 parts, among them J3 1715721, Q7 SiS443DN, Q8 MMBT3904VL, U10 ADP7182ACPZN, U3 TSR3-2450N, U4 ADP5071AREZ, U5 ADP7142ACPZN, U6 ADP7142ARDZ-3.3, U7 ADP7182ACPZN, U8 ADP7142ARDZ, U9 ADP7182ACPZN

Commit message: GERBER
Parts:
- U10, U7, U9: value ADP7182ACPZN -> ADP7182ACPZN-R7
- U5: value ADP7142ACPZN -> ADP7142ARDZ-R7; footprint Package_CSP:LFCSP-6-1EP_2x2mm_P0.65mm_EP1x1.6mm -> Package_SO:SOIC-8-1EP_3.9x4.9mm_P1.27mm_EP2.29x3mm; symbol MADC_ARTY:ADP7142ACPZN -> Regulator_Linear:ADP7142ARDZ
- U8: value ADP7142ARDZ -> ADP7142ARDZ-R7
Connections:
- net +16V: now also U5.2 (VOUT)
- net +18V: now also U5.5 (EN), U5.7 (VIN), U5.8 (VIN); no longer U5.4 (EN), U5.6 (VIN)
- net GND: now also U5.4 (GND), U5.9 (GND); no longer U5.3 (GND), U5.7 (EPAD)
- net at R18.2, R19.1: now also U5.3 (SENSE/ADJ); no longer U5.2 (ADJ)
Changed lines of the file:
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@@
 	)
 	(junction
-		(at 67.31 52.07)
+		(at 106.68 39.37)
 		(diameter 0)
 		(color 0 0 0 0)
 	)
 	(junction
-		(at 105.41 39.37)
+		(at 67.31 52.07)
 		(diameter 0)
 		(color 0 0 0 0)
@@
 	)
 	(junction
-		(at 107.95 39.37)
-		(diameter 0)
-		(color 0 0 0 0)
-	)
-	(junction
 		(at 213.36 109.22)
 		(diameter 0)
@@
 	)
 	(no_connect
-		(at 96.52 29.21)
+		(at 116.84 27.94)
 	)
 	(no_connect
@@
 	(wire
 		(pts
+			(xy 106.68 39.37) (xy 121.92 39.37)
+		)
+		(stroke
+			(width 0)
+			(type default)
+		)
+	)
+	(wire
+		(pts
 			(xy 238.76 71.12) (xy 242.57 71.12)
 		)
@@
 	(wire
 		(pts
-			(xy 96.52 25.4) (xy 95.25 25.4)
-		)
-		(stroke
-			(width 0)
-			(type default)
-		)
-	)
-	(wire
-		(pts
 			(xy 69.85 157.48) (xy 69.85 151.13)
 		)
@@
 	(wire
 		(pts
-			(xy 118.11 30.48) (xy 121.92 30.48)
+			(xy 106.68 33.02) (xy 106.68 39.37)
+		)
+		(stroke
+			(width 0)
+			(type default)
+		)
+	)
+	(wire
+		(pts
+			(xy 119.38 30.48) (xy 121.92 30.48)
 		)
 		(stroke
@@
 	(wire
 		(pts
+			(xy 96.52 27.94) (xy 95.25 27.94)
+		)
+		(stroke
+			(width 0)
+			(type default)
+		)
+	)
+	(wire
+		(pts
 			(xy 95.25 22.86) (xy 85.09 22.86)
 		)
@@
 	(wire
 		(pts
-			(xy 105.41 33.02) (xy 105.41 39.37)
-		)
-		(stroke
-			(width 0)
-			(type default)
-		)
-	)
-	(wire
-		(pts
 			(xy 66.04 36.83) (xy 67.31 36.83)
 		)
@@
 	(wire
 		(pts
-			(xy 107.95 33.02) (xy 107.95 39.37)
-		)
-		(stroke
-			(width 0)
-			(type default)
-		)
-	)
-	(wire
-		(pts
 			(xy 199.39 26.67) (xy 199.39 22.86)
 		)
@@
 	(wire
 		(pts
-			(xy 116.84 25.4) (xy 118.11 25.4)
+			(xy 116.84 25.4) (xy 119.38 25.4)
 		)
 		(stroke
@@
 	(wire
 		(pts
-			(xy 118.11 25.4) (xy 118.11 30.48)
+			(xy 119.38 25.4) (xy 119.38 30.48)
 		)
 		(stroke
@@
 	(wire
 		(pts
-			(xy 95.25 25.4) (xy 95.25 22.86)
+			(xy 95.25 22.86) (xy 95.25 27.94)
 		)
 		(stroke
@@
 	(wire
 		(pts
-			(xy 107.95 39.37) (xy 121.92 39.37)
+			(xy 85.09 39.37) (xy 106.68 39.37)
 		)
 		(stroke
@@
 	(wire
 		(pts
-			(xy 85.09 39.37) (xy 105.41 39.37)
-		)
-		(stroke
-			(width 0)
-			(type default)
-		)
-	)
-	(wire
-		(pts
 			(xy 39.37 76.2) (xy 48.26 76.2)
 		)
@@
 	(wire
 		(pts
-			(xy 105.41 39.37) (xy 107.95 39.37)
-		)
-		(stroke
-			(width 0)
-			(type default)
-		)
-	)
-	(wire
-		(pts
 			(xy 39.37 91.44) (xy 39.37 96.52)
 		)
@@
 			)
 		)
-		(property "Value" "ADP7182ACPZN"
+		(property "Value" "ADP7182ACPZN-R7"
 			(at 172.72 17.78 0)
 			(effects
@@
 			)
 		)
-		(property "Value" "ADP7182ACPZN"
+		(property "Value" "ADP7182ACPZN-R7"
 			(at 224.79 161.29 0)
 			(effects
@@
 			)
 		)
-		(property "Value" "ADP7142ARDZ"
+		(property "Value" "ADP7142ARDZ-R7"
 			(at 224.79 55.88 0)
 			(effects
@@
 	)
 	(symbol
-		(lib_id "MADC_ARTY:ADP7142ACPZN")
+		(lib_id "Regulator_Linear:ADP7142ARDZ")
 		(at 106.68 25.4 0)
 		(unit 1)
@@
 			)
 		)
-		(property "Value" "ADP7142ACPZN"
+		(property "Value" "ADP7142ARDZ-R7"
 			(at 106.68 17.78 0)
 			(effects
@@
 			)
 		)
-		(property "Footprint" "Package_CSP:LFCSP-6-1EP_2x2mm_P0.65mm_EP1x1.6mm"
+		(property "Footprint" "Package_SO:SOIC-8-1EP_3.9x4.9mm_P1.27mm_EP2.29x3mm"
 			(at 106.68 35.56 0)
 			(effects
@@
 			)
 		)
-		(property "Description" "200mA, Low Noise, CMOS Low Dropout Regulator, Positive, Adjustable"
+		(property "Description" "200mA, Low Noise, CMOS Low Dropout Regulator, Positive, Adjustable, SOIC-8"
 			(at 106.68 25.4 0)
 			(effects
@@
 		(pin "5"
 		)
+		(pin "9"
+		)
+		(pin "8"
+		)
 		(instances
 			(project ""
@@
 			)
 		)
-		(property "Value" "ADP7182ACPZN"
+		(property "Value" "ADP7182ACPZN-R7"
 			(at 224.79 119.38 0)
 			(effects
