File: Hardware/MADC_ARTY/VoltageReference.kicad_sch (KiCad schematic)
At the start: 23 parts, among them U19 OPA2192IDGKT, U20 OPA2192IDGKT, U21 ADR1399KHZ, U22 ADR1399KEZ

Commit message: GERBER
Parts:
- R70: value 2k7/1%/250mW -> 1k8/1%/250mW
- U19, U20: value OPA2192IDGKT -> OPA2192IDR
Changed lines of the file:
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@@
 			)
 		)
-		(property "Value" "2k7/1%/250mW"
+		(property "Value" "1k8/1%/250mW"
 			(at 86.36 80.0099 0)
 			(effects
@@
 			)
 		)
-		(property "Value" "OPA2192IDGKT"
+		(property "Value" "OPA2192IDR"
 			(at 23.5712 181.483 0)
 			(effects
@@
 			)
 		)
-		(property "Value" "OPA2192IDGKT"
+		(property "Value" "OPA2192IDR"
 			(at 160.782 98.298 0)
 			(effects
@@
 			)
 		)
-		(property "Value" "OPA2192IDGKT"
+		(property "Value" "OPA2192IDR"
 			(at 215.9 72.39 0)
 			(effects
@@
 			)
 		)
-		(property "Value" "OPA2192IDGKT"
+		(property "Value" "OPA2192IDR"
 			(at 45.1612 181.483 0)
 			(effects
@@
 			)
 		)
-		(property "Value" "OPA2192IDGKT"
+		(property "Value" "OPA2192IDR"
 			(at 125.73 176.53 0)
 			(effects
@@
 			)
 		)
-		(property "Value" "OPA2192IDGKT"
+		(property "Value" "OPA2192IDR"
 			(at 119.38 85.6996 0)
 			(effects
